File: blade-plate-med-no-teeth/blade-plate-med-no-teeth.kicad_pcb (KiCad board)
At the start: 2 copper layers, 37.1 x 45.1 mm, 3 parts

Commit message: Fix warnings
Other:
- rule pad_to_mask_clearance: 0.2 -> 0
